File: Hardware/MS5803-14BA_Breakout.brd (EAGLE design)
At the start: 20.3 x 17.8 mm, 18 parts, among them U1 MS5803-14BA

Commit message: changed I2C resistors to 2.2k, updated rev numbers, Moved to new jumper package
Parts:
- R1, R2: value (none) -> 2.2k; device SparkFun-Resistors:0603 -> SparkFun-Resistors:0603-RES
- SJ1: device SparkFun-Passives:SJ_3_PASTE1&2&3 -> SparkFun-Passives:PAD-JUMPER-3-NC_BY_PASTE_YES_SILK_FULL_BOX
Other:
- board text added: "v10"
- board text removed: "v01"
Changed lines of the file:
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@@
 CS</text>
 <text x="17.78" y="2.794" size="0.8128" layer="22" font="vector" ratio="15" rot="MR90" align="center-left">PS</text>
-<text x="19.558" y="0.508" size="0.8128" layer="16" font="vector" ratio="20" rot="MR270" align="center-right">v01</text>
+<text x="19.558" y="0.508" size="0.8128" layer="16" font="vector" ratio="20" rot="MR270" align="center-right">v10</text>
 </plain>
 <attributes>
@@
 <element name="U1" library="MS5803" package="MS5803" value="MS5803-14BA" x="10.16" y="11.43" smashed="yes" rot="R270">
 <attribute name="NAME" x="13.716" y="14.732" size="0.8128" layer="25" font="vector" ratio="15" rot="R270"/>
+<attribute name="PROD_ID" value="IC-12111" x="10.16" y="11.43" size="1.778" layer="27" rot="R270" display="off"/>
 </element>
 <element name="FRAME1" library="SparkFun-Aesthetics" package="CREATIVE_COMMONS" value="FRAME-LETTER" x="0" y="-8.89"/>
@@
 <attribute name="PROD_ID" value="CAP-00810" x="7.366" y="6.35" size="1.778" layer="27" rot="R180" display="off"/>
 </element>
-<element name="R1" library="SparkFun-Resistors" package="0603" value="" x="5.08" y="12.954" rot="R180">
-<attribute name="PROD_ID" value="RES-07857" x="5.08" y="12.954" size="1.778" layer="27" rot="R180" display="off"/>
-</element>
-<element name="R2" library="SparkFun-Resistors" package="0603" value="" x="5.08" y="11.176" rot="R180">
-<attribute name="PROD_ID" value="RES-07857" x="5.08" y="11.176" size="1.778" layer="27" rot="R180" display="off"/>
-</element>
-<element name="SJ1" library="SparkFun-Passives" package="SJ_3_PASTE1&amp;2&amp;3" value="" x="2.032" y="12.192" rot="R90"/>
+<element name="R1" library="SparkFun-Resistors" package="0603-RES" value="2.2k" x="5.08" y="12.954" rot="R180">
+<attribute name="PROD_ID" value="RES-08272" x="5.08" y="12.954" size="1.778" layer="27" rot="R180" display="off"/>
+<attribute name="VALUE" value="2.2k" x="5.08" y="12.954" size="1.778" layer="27" rot="R180" display="off"/>
+</element>
+<element name="R2" library="SparkFun-Resistors" package="0603-RES" value="2.2k" x="5.08" y="11.176" rot="R180">
+<attribute name="PROD_ID" value="RES-08272" x="5.08" y="11.176" size="1.778" layer="27" rot="R180" display="off"/>
+<attribute name="VALUE" value="2.2k" x="5.08" y="11.176" size="1.778" layer="27" rot="R180" display="off"/>
+</element>
+<element name="SJ1" library="SparkFun-Passives" package="PAD-JUMPER-3-NC_BY_PASTE_YES_SILK_FULL_BOX" value="" x="2.032" y="12.192" rot="R90"/>
 <element name="STANDOFF1" library="SparkFun-Electromechanical" package="STAND-OFF-TIGHT" value="STAND-OFFTIGHT" x="2.54" y="7.62"/>
 <element name="STANDOFF2" library="SparkFun-Electromechanical" package="STAND-OFF-TIGHT" value="STAND-OFFTIGHT" x="17.78" y="15.24"/>
